Commit message: modified/added files to support two zed boot

File: zed_wrapper/urdf/zedm_2.urdf (robot description, URDF)
Before this commit: robot zedm_camera_1, 7 links, 6 joints
Links:
- removed link zed_camera_center_1
- removed link zed_imu_link_1
- removed link zed_left_camera_frame_1
- removed link zed_left_camera_optical_frame_1
- removed link zed_right_camera_frame_1
- removed link zed_right_camera_optical_frame_1
- added link zed_camera_center_2; visual mesh filename=package://zed_wrapper/urdf/models/ZEDM.stl
- added link zed_imu_link_2
- added link zed_left_camera_frame_2
- added link zed_left_camera_optical_frame_2
- added link zed_right_camera_frame_2
- added link zed_right_camera_optical_frame_2
Joints:
- removed joint imu_link_joint
- removed joint zed_camera_center_joint_1
- removed joint zed_left_camera_joint_1
- removed joint zed_left_camera_optical_joint_1
- removed joint zed_right_camera_joint_1
- removed joint zed_right_camera_optical_joint_1
- added joint imu_link_joint_2: type floating, parent zed_camera_center_2, child zed_imu_link_2, origin xyz=0 0 0 rpy=0 0 0
- added joint zed_camera_center_joint_2: type fixed, parent base_link, child zed_camera_center_2, origin xyz=0.08 -0.03 0.027 rpy=0 0 0
- added joint zed_left_camera_joint_2: type fixed, parent zed_camera_center_2, child zed_left_camera_frame_2, origin xyz=0 0.03 0 rpy=0 0 0
- added joint zed_left_camera_optical_joint_2: type fixed, parent zed_left_camera_frame_2, child zed_left_camera_optical_frame_2, origin xyz=0 0 0 rpy=-1.57079632679 0.0 -1.57079632679
- added joint zed_right_camera_joint_2: type fixed, parent zed_camera_center_2, child zed_right_camera_frame_2, origin xyz=0 -0.03 0 rpy=0 0 0
- added joint zed_right_camera_optical_joint_2: type fixed, parent zed_right_camera_frame_2, child zed_right_camera_optical_frame_2, origin xyz=0 0 0 rpy=-1.57079632679 0.0 -1.57079632679

Commit message: updated zed2 urdf

File: zed_wrapper/urdf/zedm_2.urdf (robot description, URDF)
Before this commit: robot zedm_camera_2, 7 links, 6 joints
Joints:
- joint zed_camera_center_joint_2: origin xyz=0.08 -0.03 0.027 rpy=0 0.0349066 0 -> xyz=-0.08 -0.03 0.027 rpy=0 0.0349066 0
