Commit message: Added seperate zedm_1.urdf

File: zed_wrapper/urdf/zedm_1.urdf (robot description, URDF)
Before this commit: robot zedm_camera, 7 links, 6 joints
Links:
- removed link zed_camera_center
- removed link zed_imu_link
- removed link zed_left_camera_frame
- removed link zed_left_camera_optical_frame
- removed link zed_right_camera_frame
- removed link zed_right_camera_optical_frame
- added link zed_camera_center_1; visual mesh filename=package://zed_wrapper/urdf/models/ZEDM.stl
- added link zed_imu_link_1
- added link zed_left_camera_frame_1
- added link zed_left_camera_optical_frame_1
- added link zed_right_camera_frame_1
- added link zed_right_camera_optical_frame_1
Joints:
- removed joint zed_camera_center_joint
- removed joint zed_left_camera_joint
- removed joint zed_left_camera_optical_joint
- removed joint zed_right_camera_joint
- removed joint zed_right_camera_optical_joint
- added joint zed_camera_center_joint_1: type fixed, parent base_link, child zed_camera_center_1, origin xyz=0 0.085 0.03 rpy=0 0 1.57
- added joint zed_left_camera_joint_1: type fixed, parent zed_camera_center_1, child zed_left_camera_frame_1, origin xyz=0 0.03 0 rpy=0 0 0
- added joint zed_left_camera_optical_joint_1: type fixed, parent zed_left_camera_frame_1, child zed_left_camera_optical_frame_1, origin xyz=0 0 0 rpy=-1.57079632679 0.0 -1.57079632679
- added joint zed_right_camera_joint_1: type fixed, parent zed_camera_center_1, child zed_right_camera_frame_1, origin xyz=0 -0.03 0 rpy=0 0 0
- added joint zed_right_camera_optical_joint_1: type fixed, parent zed_right_camera_frame_1, child zed_right_camera_optical_frame_1, origin xyz=0 0 0 rpy=-1.57079632679 0.0 -1.57079632679
- joint imu_link_joint: child zed_imu_link -> zed_imu_link_1; parent zed_camera_center -> zed_camera_center_1

Commit message: changed urdf in order to obtain correct covariance behavior

File: zed_wrapper/urdf/zedm_1.urdf (robot description, URDF)
Before this commit: robot zedm_camera_1, 7 links, 6 joints
Joints:
- joint zed_camera_center_joint_1: origin xyz=0 0.085 0.03 rpy=0 0 1.57 -> xyz=0 0.085 0.03 rpy=0 0 0

Commit message: fixing merge overwrites

File: zed_wrapper/urdf/zedm_1.urdf (robot description, URDF)
Before this commit: robot zedm_camera_1, 7 links, 6 joints
Joints:
- joint zed_camera_center_joint_1: origin xyz=0 0.085 0.03 rpy=0 0 0 -> xyz=0 0.085 0.03 rpy=0 0 3.14159

Commit message: updated urdf for g1b2

File: zed_wrapper/urdf/zedm_1.urdf (robot description, URDF)
Before this commit: robot zedm_camera_1, 7 links, 6 joints
Joints:
- joint zed_camera_center_joint_1: origin xyz=0 0.085 0.03 rpy=0 0 3.14159 -> xyz=0 0.085 0.03 rpy=0 0.0174533 3.14159

File: zed_wrapper/urdf/zedm_2.urdf (robot description, URDF)
Before this commit: robot zedm_camera_2, 7 links, 6 joints
Joints:
- joint zed_camera_center_joint_2: origin xyz=0.08 -0.03 0.027 rpy=0 0 0 -> xyz=0.08 -0.03 0.027 rpy=0 0.0349066 0

Commit message: updated zed wrapper to find matching pointcloud and image

File: zed_wrapper/urdf/zedm_1.urdf (robot description, URDF)
Before this commit: robot zedm_camera_1, 7 links, 6 joints
Joints:
- joint zed_camera_center_joint_1: origin xyz=0 0.085 0.03 rpy=0 0.0174533 3.14159 -> xyz=-0.064 0 0.03 rpy=0 0 3.14

File: zed_wrapper/urdf/zedm_2.urdf (robot description, URDF)
Before this commit: robot zedm_camera_2, 7 links, 6 joints
Joints:
- joint zed_camera_center_joint_2: origin xyz=0.08 -0.03 0.027 rpy=0 0.0349066 0 -> xyz=0.064 0 0.03 rpy=0 0 0

Commit message: reverting to original point cloud topic and updating for g1b2 -- active drone being developed on

File: zed_wrapper/urdf/zedm_1.urdf (robot description, URDF)
Before this commit: robot zedm_camera_1, 7 links, 6 joints
Joints:
- joint zed_camera_center_joint_1: origin xyz=-0.064 0 0.03 rpy=0 0 3.14 -> xyz=0 0.085 0.03 rpy=0 0.0174533 3.14159

File: zed_wrapper/urdf/zedm_2.urdf (robot description, URDF)
Before this commit: robot zedm_camera_2, 7 links, 6 joints
Joints:
- joint zed_camera_center_joint_2: origin xyz=0.064 0 0.03 rpy=0 0 0 -> xyz=0.08 -0.03 0.027 rpy=0 0.0349066 0

Commit message: Jae's tuning changes

File: zed_wrapper/urdf/zedm_1.urdf (robot description, URDF)
Before this commit: robot zedm_camera_1, 7 links, 6 joints
Joints:
- joint zed_camera_center_joint_1: origin xyz=0 0.085 0.03 rpy=0 0.0174533 3.14159 -> xyz=0 0.085 0.03 rpy=0 -0.01745 3.14159

File: zed_wrapper/urdf/zedm_2.urdf (robot description, URDF)
Before this commit: robot zedm_camera_2, 7 links, 6 joints
Joints:
- joint zed_camera_center_joint_2: origin xyz=0.08 -0.03 0.027 rpy=0 0.0349066 0 -> xyz=0.08 -0.03 0.027 rpy=0 -0.05555549066 0

Commit message: creating branch for disney drone

File: zed_wrapper/urdf/zedm_1.urdf (robot description, URDF)
Before this commit: robot zedm_camera_1, 7 links, 6 joints
Joints:
- joint zed_camera_center_joint_1: origin xyz=0 0.085 0.03 rpy=0 0.0174533 3.14159 -> xyz=0 0.085 0.03 rpy=0 0.01745 3.14159

Commit message: tagged for demo drone Oct 14th

File: zed_wrapper/urdf/zedm_1.urdf (robot description, URDF)
Before this commit: robot zedm_camera_1, 7 links, 6 joints
Joints:
- joint zed_camera_center_joint_1: origin xyz=0 0.085 0.03 rpy=0 0.0174533 3.14159 -> xyz=0 0.085 0.03 rpy=0.1 0.0174533 0

Commit message: Revert "tagged for demo drone Oct 14th"
This reverts commit 17e1cd58ecff612a320c122446bbe1f77155f274.

File: zed_wrapper/urdf/zedm_1.urdf (robot description, URDF)
Before this commit: robot zedm_camera_1, 7 links, 6 joints
Joints:
- joint zed_camera_center_joint_1: origin xyz=0 0.085 0.03 rpy=0.1 0.0174533 0 -> xyz=0 0.085 0.03 rpy=0 0.0174533 3.14159

Commit message: demo drone updated

File: zed_wrapper/urdf/zedm_1.urdf (robot description, URDF)
Before this commit: robot zedm_camera_1, 7 links, 6 joints
Joints:
- joint zed_camera_center_joint_1: origin xyz=0 0.085 0.03 rpy=0 0.0174533 3.14159 -> xyz=0 0.085 0.03 rpy=0.0 0.0 -0.05

Commit message: adjusted urdf

File: zed_wrapper/urdf/zedm_1.urdf (robot description, URDF)
Before this commit: robot zedm_camera_1, 7 links, 6 joints
Joints:
- joint zed_camera_center_joint_1: origin xyz=0 0.085 0.03 rpy=0.0 0.0 -0.05 -> xyz=0 0.085 0.03 rpy=0.1 0.0174533 0

Commit message: enable odom_init true

File: zed_wrapper/urdf/zedm_1.urdf (robot description, URDF)
Before this commit: robot zedm_camera_1, 7 links, 6 joints
Joints:
- joint zed_camera_center_joint_1: origin xyz=0 0.085 0.03 rpy=0 0.0174533 3.14159 -> xyz=0 0.085 0.03 rpy=0 0  3.14159

File: zed_wrapper/urdf/zedm_2.urdf (robot description, URDF)
Before this commit: robot zedm_camera_2, 7 links, 6 joints
Joints:
- joint zed_camera_center_joint_2: origin xyz=0.08 -0.03 0.027 rpy=0 0.0349066 0 -> xyz=0.08 -0.03 0.027 rpy=0 0 0

Commit message: updated zedm_1.urdf: flying better

File: zed_wrapper/urdf/zedm_1.urdf (robot description, URDF)
Before this commit: robot zedm_camera_1, 7 links, 6 joints
Joints:
- joint zed_camera_center_joint_1: origin xyz=0 0.085 0.03 rpy=0.1 0.0174533 0 -> xyz=0 0.085 0.03 rpy=0.04 0.0174533 0

Commit message: calibrate~.py working; changed zed1

File: zed_wrapper/urdf/zedm_1.urdf (robot description, URDF)
Before this commit: robot zedm_camera_1, 7 links, 6 joints
Joints:
- joint zed_camera_center_joint_1: origin xyz=0 0.085 0.03 rpy=0 0.0174533 3.14159 -> xyz=0 0.085 0.03 rpy=0 0 3.14159
